Commit message: feat(gui): configure and measure offset cutting tools

File: ros2/src/mowgli_bringup/urdf/mowgli.urdf.xacro (robot description, xacro)
@@ -75,4 +75,6 @@
   <xacro:arg name="caster_x_offset"  default="0.40"/>
   <xacro:arg name="blade_radius"     default="0.09"/>
+  <xacro:arg name="blade_x_offset" default="0.0"/>
+  <xacro:arg name="blade_y_offset" default="0.0"/>
   <!-- ================================================================
        Properties (resolved from args — all shape from config)
@@ -98,4 +100,6 @@
   <xacro:property name="base_mass"        value="$(arg chassis_mass_kg)"/>
   <xacro:property name="blade_radius"     value="$(arg blade_radius)"/>
+  <xacro:property name="blade_x_offset" value="$(arg blade_x_offset)"/>
+  <xacro:property name="blade_y_offset" value="$(arg blade_y_offset)"/>
   <xacro:property name="blade_height"     value="0.01"/>
   <xacro:property name="blade_mass"       value="0.3"/>
@@ -289,6 +293,6 @@
     <parent link="base_link"/>
     <child  link="blade_link"/>
-    <!-- Blade disc centred under chassis -->
-    <origin xyz="${chassis_cx} 0 ${-wheel_radius + 0.05}" rpy="0 0 0"/>
+    <!-- Offsets from chassis centre: +X forward, +Y left. Zero preserves legacy geometry. -->
+    <origin xyz="${chassis_cx + blade_x_offset} ${blade_y_offset} ${-wheel_radius + 0.05}" rpy="0 0 0"/>
   </joint>
   <!-- ================================================================
